Commit message: Fixed errors in urdf

File: launch_config/urdf/ballast.xacro (robot description, xacro)
@@ -17,5 +17,5 @@
             </inertial>
         </link>
-        <joint name="${name}" type="fixed">
+        <joint name="${name}_joint" type="fixed">
             <origin xyz="${xyz}"/>
             <parent link="base_link"/>

File: launch_config/urdf/mallard_main.xacro (robot description, xacro)
@@ -9,11 +9,8 @@
   <!-- Thrusters components & constants -->
   <xacro:property name="PI" value="3.1415926535897931"/>
-  <xacro:property name="tr1" value=".02" />
-  <xacro:property name="tl1" value=".1" />
-  <xacro:property name="tr2" value=".047" />
-  <xacro:property name="tl2" value=".045" />
-  <gazebo reference="base_link">
-      <material>Gazebo/Blue</material>
-  </gazebo>
+  <xacro:property name="thruster_length_1" value=".1" />
+  <xacro:property name="thruster_length_2" value=".045" />
+  <xacro:property name="thruster_radius_2" value=".047" />
+  <xacro:property name="thruster_radius_1" value=".02" />
   <link name="base_link">
       <!-- Channels (aluminum connecting elements) -->
@@ -78,12 +75,12 @@
 	</xacro:lidar>
   <!-- Ballast -->
-  <xacro:ballast name="ballast_1" mass="0.14" xyz=" 0.225 -0.25 0.076" rpy="${PI/2} 0 0"/>
+  <xacro:ballast name="ballast_1" mass="0.14" xyz="0.225 -0.25 0.076" rpy="${PI/2} 0 0"/>
   <xacro:ballast name="ballast_2" mass="0.02" xyz="-0.225 -0.25 0.076" rpy="${PI/2} 0 0"/>
   <!-- Forward thrusters -->
-  <xacro:thruster_link name="x_thr_left"   xyz="${(tl1/2)-0.188}  0.207 -0.041" rpy="0 ${-PI/2} 0"/>
-  <xacro:thruster_link name="x_thr_right"  xyz="${(tl1/2)-0.188} -0.207 -0.041" rpy="0 ${-PI/2} 0"/>
+  <xacro:thruster_link name="x_thr_left"   xyz="${(thruster_length_1/2)-0.188} 0.207 -0.041" rpy="0 ${-PI/2} 0"/>
+  <xacro:thruster_link name="x_thr_right"  xyz="${(thruster_length_1/2)-0.188} -0.207 -0.041" rpy="0 ${-PI/2} 0"/>
   <!-- Side thrusters -->
-  <xacro:thruster_link name="y_thr_right"   xyz=" 0.233 ${0.114-(tl1/2)} -0.041" rpy="0 ${PI/2} ${PI/2}"/>
-  <xacro:thruster_link name="y_thr_left"  xyz="-0.233 ${0.114-(tl1/2)} -0.041" rpy="0 ${PI/2} ${PI/2}"/>
+  <xacro:thruster_link name="y_thr_right"   xyz="0.233 ${0.114-(thruster_length_1/2)} -0.041" rpy="0 ${PI/2} ${PI/2}"/>
+  <xacro:thruster_link name="y_thr_left"  xyz="-0.233 ${0.114-(thruster_length_1/2)} -0.041" rpy="0 ${PI/2} ${PI/2}"/>
   <!-- FreeFloating plugin -->
   <gazebo>
@@ -91,5 +88,5 @@
           <switchService>switch</switchService>
           <updateRate>100</updateRate>
-          <link>base_link</link>
+          <link>mallard_link</link>
                 <!-- THRUST CONTROL -->
                 <!--    these two thrusters are actually orientable, so the map should not be hard-coded

File: launch_config/urdf/thruster.xacro (robot description, xacro)
@@ -2,5 +2,5 @@
 <robot xmlns:xacro="http://www.ros.org/wiki/xacro" name="mallard">
     <xacro:macro name="thruster_link" params="name xyz rpy">
-      <joint name="${name}" type="revolute">
+      <joint name="${name}_joint" type="revolute">
           <parent link="base_link"/>
           <child link="${name}"/>
@@ -13,5 +13,5 @@
           <visual name="${name}_1">
               <geometry>
-                  <cylinder length="${tl1}" radius="${tr1}"/>
+                  <cylinder length="${thruster_length_1}" radius="${thruster_radius_1}"/>
               </geometry>
               <material name="blue">
@@ -20,7 +20,7 @@
           </visual>
           <visual name="${name}_2">
-              <origin xyz="0 0 ${tl2/4}"/>
+              <origin xyz="0 0 ${thruster_length_2/4}"/>
               <geometry>
-                  <cylinder length="${tl2}" radius="${tr2}"/>
+                  <cylinder length="${thruster_length_2}" radius="${thruster_radius_2}"/>
               </geometry>
               <material name="blue">
